File: USBCerial.sch (KiCad schematic (older format))
At the start: 3 parts, among them J1 USB_C, U1 CH340C

Commit message: ifxed the footprints
Parts:
- C1: footprint Capacitor_SMD:C_0603_1608Metric -> Capacitor_SMD:C_0603_1608Metric_Pad1.08x0.95mm_HandSolder
Connections:
- wire segments 12 -> 11
Changed lines of the file:
@@
 L Device:C C1
 U 1 1 60D1A9EC
-P 3200 2750
-F 0 "C1" H 3315 2796 50  0000 L CNN
-F 1 "0.1uF" H 3315 2705 50  0000 L CNN
-F 2 "Capacitor_SMD:C_0603_1608Metric" H 3238 2600 50  0001 C CNN
-F 3 "~" H 3200 2750 50  0001 C CNN
-	1    3200 2750
+P 3200 2700
+F 0 "C1" H 3315 2746 50  0000 L CNN
+F 1 "0.1uF" H 3315 2655 50  0000 L CNN
+F 2 "Capacitor_SMD:C_0603_1608Metric_Pad1.08x0.95mm_HandSolder" H 3238 2550 50  0001 C CNN
+F 3 "~" H 3200 2700 50  0001 C CNN
+	1    3200 2700
 	1    0    0    -1
 $EndComp
@@
 	3200 2500 3200 2400
 Wire Wire Line
-	3200 2600 3200 2500
+	3200 2550 3200 2500
 Connection ~ 3200 2500
 $Comp
 L power:GND #PWR0103
 U 1 1 60D22F42
-P 3200 2950
-F 0 "#PWR0103" H 3200 2700 50  0001 C CNN
-F 1 "GND" H 3205 2777 50  0000 C CNN
-F 2 "" H 3200 2950 50  0001 C CNN
-F 3 "" H 3200 2950 50  0001 C CNN
-	1    3200 2950
+P 3200 2850
+F 0 "#PWR0103" H 3200 2600 50  0001 C CNN
+F 1 "GND" H 3205 2677 50  0000 C CNN
+F 2 "" H 3200 2850 50  0001 C CNN
+F 3 "" H 3200 2850 50  0001 C CNN
+	1    3200 2850
 	1    0    0    -1
 $EndComp
-Wire Wire Line
-	3200 2900 3200 2950
 $Comp
 L power:GND #PWR0104
