File: USBCereal.sch (KiCad schematic (older format))
At the start: 14 parts, among them J1 USB_C, J2 Conn_01x06, U1 XC6206P332MR, U2 CH340C

Commit message: Complete the PCB, ficed spelling errors
Parts:
- D1, D2: footprint LED_SMD:LED_0603_1608Metric_Castellated -> LED_SMD:LED_0603_1608Metric_Pad1.05x0.95mm_HandSolder
Connections:
- net shield: no longer names the net of J1.S1 (SHIELD)
- no-connect marks 7 -> 8
Changed lines of the file:
@@
 	1900 1800 1750 1800
 Connection ~ 1900 1800
-Text GLabel 850  2500 3    50   Input ~ 0
-shield
 $Comp
 L power:+5V #PWR03
@@
 Wire Wire Line
 	1750 1000 2950 1000
-$Comp
-L Connector:USB_C_Receptacle_USB2.0 J1
-U 1 1 60D11074
-P 1150 1600
-F 0 "J1" H 1150 2450 50  0000 C CNN
-F 1 "USB_C" H 1150 2350 50  0000 C CNN
-F 2 "Connector_USB:USB_C_Receptacle_GCT_USB4085" H 1300 1600 50  0001 C CNN
-F 3 "https://www.usb.org/sites/default/files/documents/usb_type-c.zip" H 1300 1600 50  0001 C CNN
-F 4 "2137160001" H 1150 1600 50  0001 C CNN "Part Number"
-	1    1150 1600
-	1    0    0    -1
-$EndComp
 NoConn ~ 1750 2100
 NoConn ~ 1750 2200
@@
 F 0 "D1" V 7550 1475 50  0000 R CNN
 F 1 "LED_Small" H 7650 1250 50  0000 R CNN
-F 2 "LED_SMD:LED_0603_1608Metric_Castellated" V 7475 1350 50  0001 C CNN
+F 2 "LED_SMD:LED_0603_1608Metric_Pad1.05x0.95mm_HandSolder" V 7475 1350 50  0001 C CNN
 F 3 "~" V 7475 1350 50  0001 C CNN
 F 4 "19-217/BHC-ZL1M2RY/3T" V 7475 1350 50  0001 C CNN "Part Number"
@@
 F 0 "D2" V 7875 1475 50  0000 R CNN
 F 1 "LED_Small" H 7975 1250 50  0000 R CNN
-F 2 "LED_SMD:LED_0603_1608Metric_Castellated" V 7800 1350 50  0001 C CNN
+F 2 "LED_SMD:LED_0603_1608Metric_Pad1.05x0.95mm_HandSolder" V 7800 1350 50  0001 C CNN
 F 3 "~" V 7800 1350 50  0001 C CNN
 F 4 "19-217/BHC-ZL1M2RY/3T" V 7800 1350 50  0001 C CNN "Part Number"
@@
 Text Notes 8725 600  2    50   ~ 0
 Output Header
+$Comp
+L Connector:USB_C_Receptacle_USB2.0 J1
+U 1 1 60D11074
+P 1150 1600
+F 0 "J1" H 1150 2450 50  0000 C CNN
+F 1 "USB_C" H 1150 2350 50  0000 C CNN
+F 2 "Connector_USB:USB_C_Receptacle_GCT_USB4085" H 1300 1600 50  0001 C CNN
+F 3 "https://www.usb.org/sites/default/files/documents/usb_type-c.zip" H 1300 1600 50  0001 C CNN
+F 4 "2137160001" H 1150 1600 50  0001 C CNN "Part Number"
+	1    1150 1600
+	1    0    0    -1
+$EndComp
+NoConn ~ 850  2500
 $EndSCHEMATC

Commit message: Finished PCB, generated fabrication files
Parts:
- C1, C2, C3: LCSC (none) -> CL10A105KB8NNNC
- D1, D2: LCSC (none) -> 19-217/BHC-ZL1M2RY/3T
- J1: footprint Connector_USB:USB_C_Receptacle_GCT_USB4085 -> Connector_USB:USB_C_Receptacle_HRO_TYPE-C-31-M-12; LCSC (none) -> C165948
- R1, R2: LCSC (none) -> 0603WAF5101T5E
- R3, R4: value 51 -> 47R; LCSC (none) -> 0603WAF470JT5E
- U1: LCSC (none) -> C5446
- U2: LCSC (none) -> C84681
Changed lines of the file:
@@
 F 2 "Package_SO:SOIC-16_3.9x9.9mm_P1.27mm" H 6600 1325 50  0001 L CNN
 F 3 "https://datasheet.lcsc.com/szlcsc/Jiangsu-Qin-Heng-CH340C_C84681.pdf" H 6200 2675 50  0001 C CNN
+F 4 "C84681" H 6550 1875 50  0001 C CNN "LCSC"
 	1    6550 1875
 	1    0    0    -1
@@
 F 2 "Package_TO_SOT_SMD:SOT-23" H 4500 1225 50  0001 C CIN
 F 3 "https://www.torexsemi.com/file/xc6206/XC6206.pdf" H 4500 1000 50  0001 C CNN
+F 4 "C5446" H 4500 1000 50  0001 C CNN "LCSC"
 	1    4500 1000
 	1    0    0    -1
@@
 F 3 "~" H 3950 1250 50  0001 C CNN
 F 4 "CL10A105KB8NNNC" H 3950 1250 50  0001 C CNN "Part Number"
+F 5 "CL10A105KB8NNNC" H 3950 1250 50  0001 C CNN "LCSC"
 	1    3950 1250
 	1    0    0    -1
@@
 F 3 "~" H 5000 1250 50  0001 C CNN
 F 4 "CL10A105KB8NNNC" H 5000 1250 50  0001 C CNN "Part Number"
+F 5 "CL10A105KB8NNNC" H 5000 1250 50  0001 C CNN "LCSC"
 	1    5000 1250
 	1    0    0    -1
@@
 F 3 "~" H 2350 1400 50  0001 C CNN
 F 4 "0603WAF5101T5E" H 2350 1400 50  0001 C CNN "Part Number"
+F 5 "0603WAF5101T5E" H 2350 1400 50  0001 C CNN "LCSC"
 	1    2350 1400
 	1    0    0    -1
@@
 F 3 "~" H 2650 1400 50  0001 C CNN
 F 4 "0603WAF5101T5E" H 2650 1400 50  0001 C CNN "Part Number"
+F 5 "0603WAF5101T5E" H 2650 1400 50  0001 C CNN "LCSC"
 	1    2650 1400
 	1    0    0    -1
@@
 F 3 "~" H 2950 1250 50  0001 C CNN
 F 4 "CL10A105KB8NNNC" H 2950 1250 50  0001 C CNN "Part Number"
+F 5 "CL10A105KB8NNNC" H 2950 1250 50  0001 C CNN "LCSC"
 	1    2950 1250
 	1    0    0    -1
@@
 P 7475 1025
 F 0 "R3" H 7534 1071 50  0000 L CNN
-F 1 "51" H 7534 980 50  0000 L CNN
+F 1 "47R" H 7534 980 50  0000 L CNN
 F 2 "Resistor_SMD:R_0603_1608Metric_Pad0.98x0.95mm_HandSolder" H 7475 1025 50  0001 C CNN
 F 3 "~" H 7475 1025 50  0001 C CNN
 F 4 "0603WAF470JT5E" H 7475 1025 50  0001 C CNN "Part Number"
+F 5 "0603WAF470JT5E" H 7475 1025 50  0001 C CNN "LCSC"
 	1    7475 1025
 	1    0    0    -1
@@
 P 7800 1025
 F 0 "R4" H 7859 1071 50  0000 L CNN
-F 1 "51" H 7859 980 50  0000 L CNN
+F 1 "47R" H 7859 980 50  0000 L CNN
 F 2 "Resistor_SMD:R_0603_1608Metric_Pad0.98x0.95mm_HandSolder" H 7800 1025 50  0001 C CNN
 F 3 "~" H 7800 1025 50  0001 C CNN
 F 4 "0603WAF470JT5E" H 7800 1025 50  0001 C CNN "Part Number"
+F 5 "0603WAF470JT5E" H 7800 1025 50  0001 C CNN "LCSC"
 	1    7800 1025
 	1    0    0    -1
@@
 F 3 "~" V 7475 1350 50  0001 C CNN
 F 4 "19-217/BHC-ZL1M2RY/3T" V 7475 1350 50  0001 C CNN "Part Number"
+F 5 "19-217/BHC-ZL1M2RY/3T" H 7475 1350 50  0001 C CNN "LCSC"
 	1    7475 1350
 	0    -1   -1   0
@@
 F 3 "~" V 7800 1350 50  0001 C CNN
 F 4 "19-217/BHC-ZL1M2RY/3T" V 7800 1350 50  0001 C CNN "Part Number"
+F 5 "19-217/BHC-ZL1M2RY/3T" H 7800 1350 50  0001 C CNN "LCSC"
 	1    7800 1350
 	0    -1   -1   0
@@
 Text Notes 8725 600  2    50   ~ 0
 Output Header
+NoConn ~ 850  2500
 $Comp
 L Connector:USB_C_Receptacle_USB2.0 J1
@@
 F 0 "J1" H 1150 2450 50  0000 C CNN
 F 1 "USB_C" H 1150 2350 50  0000 C CNN
-F 2 "Connector_USB:USB_C_Receptacle_GCT_USB4085" H 1300 1600 50  0001 C CNN
+F 2 "Connector_USB:USB_C_Receptacle_HRO_TYPE-C-31-M-12" H 1300 1600 50  0001 C CNN
 F 3 "https://www.usb.org/sites/default/files/documents/usb_type-c.zip" H 1300 1600 50  0001 C CNN
 F 4 "2137160001" H 1150 1600 50  0001 C CNN "Part Number"
+F 5 "C165948" H 1150 1600 50  0001 C CNN "LCSC"
 	1    1150 1600
 	1    0    0    -1
 $EndComp
-NoConn ~ 850  2500
 $EndSCHEMATC

Commit message: finalise fabrication files, read for JLCPCB order
Parts:
- C1: Part Number CL10A105KB8NNNC -> CC0603KRX7R9BB104
Changed lines of the file:
@@
 F 2 "Capacitor_SMD:C_0603_1608Metric_Pad1.08x0.95mm_HandSolder" H 2950 1250 50  0001 C CNN
 F 3 "~" H 2950 1250 50  0001 C CNN
-F 4 "CL10A105KB8NNNC" H 2950 1250 50  0001 C CNN "Part Number"
+F 4 "CC0603KRX7R9BB104" H 2950 1250 50  0001 C CNN "Part Number"
 F 5 "CL10A105KB8NNNC" H 2950 1250 50  0001 C CNN "LCSC"
 	1    2950 1250

Commit message: update libraries and generate the ibom
Parts:
- U2: symbol USBCerial:CH340C -> USBCereal:CH340C
Changed lines of the file:
@@
 USB_D-
 $Comp
-L USBCerial:CH340C U2
+L USBCereal:CH340C U2
 U 1 1 60D09F5C
 P 6550 1875
